File: Spannungsversorgung.sch (KiCad schematic (older format))
At the start: 0 parts

Commit message: Datenblätter hinzufügen und anschlüsse beschriften
Parts:
- added C? (x2): 100uF, symbol Device:C
- added C? (x2): 330uF, symbol Device:C
- added D? (x2): 1N5817, Diode_THT:D_DO-41_SOD81_P10.16mm_Horizontal, symbol Diode:1N5817
- added J?: Screw_Terminal_01x02, symbol Connector:Screw_Terminal_01x02
- added L? (x2): 330uH, symbol Device:L
- added U?: LM2575-3.3BT, Package_TO_SOT_THT:TO-220-5_Vertical, symbol Regulator_Switching:LM2575-3.3BT
- added U?: LM2575-5.0BT, Package_TO_SOT_THT:TO-220-5_Vertical, symbol Regulator_Switching:LM2575-5.0BT
Connections:
- new net: D?.1 (K), L?.2, U?.2 (OUT) (x2)
- new net +12V: C?.1, C?.1, J?.1 (Pin_1), U?.1 (VIN), U?.1 (VIN)
- new net 3.3V: C?.1, L?.1, U?.4 (FB)
- new net 5V: C?.1, L?.1, U?.4 (FB)
- new net GND: C?.2, C?.2, C?.2, C?.2, D?.2 (A), D?.2 (A), J?.2 (Pin_2), U?.3 (GND), U?.3 (GND), U?.5 (~ON~/OFF), U?.5 (~ON~/OFF)
