File: Anschlüsse.sch (KiCad schematic (older format))
At the start: 1 part, among them J1 Conn_02x16_Odd_Even

Commit message: Datenblätter hinzufügen und anschlüsse beschriften
Parts:
- added J?: Screw_Terminal_01x02, symbol Connector:Screw_Terminal_01x02
Connections:
- net 3.3V: now reaches J1.1 (Pin_1)
- net 5V: now reaches J1.2 (Pin_2)
- new net 12V: J?.1 (Pin_1)
- new net GND: J?.2 (Pin_2)
Changed lines of the file:
@@
 $Descr A4 11693 8268
 encoding utf-8
-Sheet 4 5
+Sheet 4 6
 Title ""
 Date ""
@@
 	1    0    0    -1
 $EndComp
+Text HLabel 4700 2600 0    50   Input ~ 0
+3.3V
+Text HLabel 5750 2600 2    50   Input ~ 0
+5V
+Text HLabel 6900 4400 0    50   Input ~ 0
+12V
+Text HLabel 6900 4500 0    50   Input ~ 0
+GND
+$Comp
+L Connector:Screw_Terminal_01x02 J?
+U 1 1 5FC65916
+P 7400 4400
+F 0 "J?" H 7480 4392 50  0000 L CNN
+F 1 "Screw_Terminal_01x02" H 7480 4301 50  0000 L CNN
+F 2 "" H 7400 4400 50  0001 C CNN
+F 3 "~" H 7400 4400 50  0001 C CNN
+	1    7400 4400
+	1    0    0    -1
+$EndComp
+Wire Wire Line
+	6900 4500 7100 4500
+$Comp
+L power:GND #PWR?
+U 1 1 5FC66604
+P 7100 4650
+F 0 "#PWR?" H 7100 4400 50  0001 C CNN
+F 1 "GND" H 7105 4477 50  0000 C CNN
+F 2 "" H 7100 4650 50  0001 C CNN
+F 3 "" H 7100 4650 50  0001 C CNN
+	1    7100 4650
+	1    0    0    -1
+$EndComp
+Wire Wire Line
+	7100 4650 7100 4500
+Connection ~ 7100 4500
+Wire Wire Line
+	7100 4500 7200 4500
+Wire Wire Line
+	6900 4400 7200 4400
+Wire Wire Line
+	5500 2600 5750 2600
+Wire Wire Line
+	5000 2600 4700 2600
 $EndSCHEMATC

Commit message: i did everithing
Parts:
- removed J1: Conn_02x16_Odd_Even, Connector_PinSocket_2.54mm:PinSocket_2x16_P2.54mm_Vertical, symbol Connector_Generic:Conn_02x16_Odd_Even
- removed J?: Screw_Terminal_01x02, symbol Connector:Screw_Terminal_01x02
- added J3: Conn_01x16_Male, Connector_PinHeader_2.00mm:PinHeader_1x16_P2.00mm_Vertical_SMD_Pin1Left, symbol Connector:Conn_01x16_Male
Connections:
- net GND: now also J3.12 (Pin_12)
- new net +12V: J3.1 (Pin_1)
- new net +3V3: J3.11 (Pin_11)
- new net +5V: J3.3 (Pin_3)
- new net Rx: J3.9 (Pin_9)
- new net SCL: J3.6 (Pin_6)
- new net SDA: J3.7 (Pin_7)
- new net SD_D0: J3.14 (Pin_14)
- new net SD_DI: J3.15 (Pin_15)
- new net SD_SCK: J3.13 (Pin_13)
- new net SD_SS: J3.16 (Pin_16)
- new net SENSOR_VN: J3.5 (Pin_5)
- new net SENSOR_VP: J3.4 (Pin_4)
- new net TX: J3.8 (Pin_8)
- no-connect marks 0 -> 2
Changed lines of the file:
@@
 $Descr A4 11693 8268
 encoding utf-8
-Sheet 4 6
+Sheet 6 6
 Title ""
 Date ""
@@
 Comment4 ""
 $EndDescr
+Text HLabel 6200 3350 3    50   Input ~ 0
+SDA
+Text HLabel 6300 3350 3    50   Input ~ 0
+SCL
+Text HLabel 5600 3350 3    50   Input ~ 0
+SD_SCK
+Text HLabel 5400 3350 3    50   Input ~ 0
+SD_DI
+Text HLabel 5500 3350 3    50   Input ~ 0
+SD_D0
+Text HLabel 5300 3350 3    50   Input ~ 0
+SD_SS
+Text HLabel 6100 3350 3    50   Input ~ 0
+TX
+Text HLabel 6000 3350 3    50   Input ~ 0
+Rx
+Text HLabel 7550 1350 0    50   Input ~ 0
+GND
+Text HLabel 8450 1350 2    50   Input ~ 0
+12V
 $Comp
-L Connector_Generic:Conn_02x16_Odd_Even J1
-U 1 1 5FB46027
-P 5200 3300
-F 0 "J1" H 5250 4217 50  0000 C CNN
-F 1 "Conn_02x16_Odd_Even" H 5250 4126 50  0000 C CNN
-F 2 "Connector_PinSocket_2.54mm:PinSocket_2x16_P2.54mm_Vertical" H 5200 3300 50  0001 C CNN
-F 3 "~" H 5200 3300 50  0001 C CNN
-	1    5200 3300
-	1    0    0    -1
-$EndComp
-Text HLabel 4700 2600 0    50   Input ~ 0
-3.3V
-Text HLabel 5750 2600 2    50   Input ~ 0
-5V
-Text HLabel 6900 4400 0    50   Input ~ 0
-12V
-Text HLabel 6900 4500 0    50   Input ~ 0
-GND
-$Comp
-L Connector:Screw_Terminal_01x02 J?
-U 1 1 5FC65916
-P 7400 4400
-F 0 "J?" H 7480 4392 50  0000 L CNN
-F 1 "Screw_Terminal_01x02" H 7480 4301 50  0000 L CNN
-F 2 "" H 7400 4400 50  0001 C CNN
-F 3 "~" H 7400 4400 50  0001 C CNN
-	1    7400 4400
+L power:GND #PWR049
+U 1 1 5FFF286B
+P 7700 1350
+F 0 "#PWR049" H 7700 1100 50  0001 C CNN
+F 1 "GND" H 7705 1177 50  0000 C CNN
+F 2 "" H 7700 1350 50  0001 C CNN
+F 3 "" H 7700 1350 50  0001 C CNN
+	1    7700 1350
 	1    0    0    -1
 $EndComp
 Wire Wire Line
-	6900 4500 7100 4500
+	7700 1350 7550 1350
 $Comp
-L power:GND #PWR?
-U 1 1 5FC66604
-P 7100 4650
-F 0 "#PWR?" H 7100 4400 50  0001 C CNN
-F 1 "GND" H 7105 4477 50  0000 C CNN
-F 2 "" H 7100 4650 50  0001 C CNN
-F 3 "" H 7100 4650 50  0001 C CNN
-	1    7100 4650
+L power:+12V #PWR051
+U 1 1 5FFF3450
+P 8350 1350
+F 0 "#PWR051" H 8350 1200 50  0001 C CNN
+F 1 "+12V" H 8365 1523 50  0000 C CNN
+F 2 "" H 8350 1350 50  0001 C CNN
+F 3 "" H 8350 1350 50  0001 C CNN
+	1    8350 1350
+	-1   0    0    1
+$EndComp
+Wire Wire Line
+	8350 1350 8450 1350
+$Comp
+L power:GND #PWR046
+U 1 1 5FFF3FA3
+P 5700 3350
+F 0 "#PWR046" H 5700 3100 50  0001 C CNN
+F 1 "GND" H 5705 3177 50  0000 C CNN
+F 2 "" H 5700 3350 50  0001 C CNN
+F 3 "" H 5700 3350 50  0001 C CNN
+	1    5700 3350
 	1    0    0    -1
 $EndComp
+$Comp
+L power:+12V #PWR050
+U 1 1 5FFF43D1
+P 7700 3250
+F 0 "#PWR050" H 7700 3100 50  0001 C CNN
+F 1 "+12V" H 7715 3423 50  0000 C CNN
+F 2 "" H 7700 3250 50  0001 C CNN
+F 3 "" H 7700 3250 50  0001 C CNN
+	1    7700 3250
+	1    0    0    -1
+$EndComp
+$Comp
+L Connector:Conn_01x16_Male J3
+U 1 1 5FD40501
+P 6100 3150
+F 0 "J3" V 5935 3078 50  0000 C CNN
+F 1 "Conn_01x16_Male" V 6026 3078 50  0000 C CNN
+F 2 "Connector_PinHeader_2.00mm:PinHeader_1x16_P2.00mm_Vertical_SMD_Pin1Left" H 6100 3150 50  0001 C CNN
+F 3 "~" H 6100 3150 50  0001 C CNN
+	1    6100 3150
+	0    1    1    0
+$EndComp
+Text HLabel 6400 3350 3    50   Input ~ 0
+SENSOR_VN
+Text HLabel 6500 3350 3    50   Input ~ 0
+SENSOR_VP
+$Comp
+L power:+3.3V #PWR047
+U 1 1 5FD44140
+P 5800 3350
+F 0 "#PWR047" H 5800 3200 50  0001 C CNN
+F 1 "+3.3V" H 5815 3523 50  0000 C CNN
+F 2 "" H 5800 3350 50  0001 C CNN
+F 3 "" H 5800 3350 50  0001 C CNN
+	1    5800 3350
+	-1   0    0    1
+$EndComp
+$Comp
+L power:+5V #PWR048
+U 1 1 5FD44777
+P 6600 3350
+F 0 "#PWR048" H 6600 3200 50  0001 C CNN
+F 1 "+5V" H 6615 3523 50  0000 C CNN
+F 2 "" H 6600 3350 50  0001 C CNN
+F 3 "" H 6600 3350 50  0001 C CNN
+	1    6600 3350
+	-1   0    0    1
+$EndComp
 Wire Wire Line
-	7100 4650 7100 4500
-Connection ~ 7100 4500
+	6800 3350 7700 3350
 Wire Wire Line
-	7100 4500 7200 4500
-Wire Wire Line
-	6900 4400 7200 4400
-Wire Wire Line
-	5500 2600 5750 2600
-Wire Wire Line
-	5000 2600 4700 2600
+	7700 3350 7700 3250
+$Comp
+L power:+3.3V #PWR053
+U 1 1 5FD45FA7
+P 8550 1900
+F 0 "#PWR053" H 8550 1750 50  0001 C CNN
+F 1 "+3.3V" H 8565 2073 50  0000 C CNN
+F 2 "" H 8550 1900 50  0001 C CNN
+F 3 "" H 8550 1900 50  0001 C CNN
+	1    8550 1900
+	1    0    0    -1
+$EndComp
+$Comp
+L power:+5V #PWR052
+U 1 1 5FD45FAD
+P 8350 1900
+F 0 "#PWR052" H 8350 1750 50  0001 C CNN
+F 1 "+5V" H 8365 2073 50  0000 C CNN
+F 2 "" H 8350 1900 50  0001 C CNN
+F 3 "" H 8350 1900 50  0001 C CNN
+	1    8350 1900
+	1    0    0    -1
+$EndComp
+Text HLabel 8350 1900 0    50   Input ~ 0
+5V
+Text HLabel 8550 1900 2    50   Input ~ 0
+3V3
+NoConn ~ 5900 3350
+NoConn ~ 6700 3350
 $EndSCHEMATC

Commit message: smal fixes
Parts:
- J3: footprint Connector_PinHeader_2.00mm:PinHeader_1x16_P2.00mm_Vertical_SMD_Pin1Left -> Connector_PinHeader_2.54mm:PinHeader_1x16_P2.54mm_Vertical_SMD_Pin1Left
Changed lines of the file:
@@
 F 0 "J3" V 5935 3078 50  0000 C CNN
 F 1 "Conn_01x16_Male" V 6026 3078 50  0000 C CNN
-F 2 "Connector_PinHeader_2.00mm:PinHeader_1x16_P2.00mm_Vertical_SMD_Pin1Left" H 6100 3150 50  0001 C CNN
+F 2 "Connector_PinHeader_2.54mm:PinHeader_1x16_P2.54mm_Vertical_SMD_Pin1Left" H 6100 3150 50  0001 C CNN
 F 3 "~" H 6100 3150 50  0001 C CNN
 	1    6100 3150

Commit message: Add CAD
Parts:
- removed J3: Conn_01x16_Male, Connector_PinHeader_2.54mm:PinHeader_1x16_P2.54mm_Vertical_SMD_Pin1Left, symbol Connector:Conn_01x16_Male
- added J3: Conn_02x08_Odd_Even, EZ-PY32:HTSS-108-01-YY-DV, symbol Connector_Generic:Conn_02x08_Odd_Even
Connections:
- net +12V: now also J3.9 (Pin_9)
- net +3V3: now also J3.10 (Pin_10)
- net +5V: now also J3.15 (Pin_15)
- net GND: now also J3.6 (Pin_6)
- net Rx: now also J3.12 (Pin_12)
- net SCL: now also J3.4 (Pin_4)
- net SDA: now also J3.2 (Pin_2)
- net SD_D0: now also J3.5 (Pin_5)
- net SD_DI: now also J3.3 (Pin_3)
- net SD_SCK: now also J3.7 (Pin_7)
- net SD_SS: now also J3.1 (Pin_1)
- net SENSOR_VN: now also J3.11 (Pin_11)
- net SENSOR_VP: now also J3.13 (Pin_13)
- net TX: now also J3.14 (Pin_14)
Changed lines of the file:
@@
 Comment4 ""
 $EndDescr
-Text HLabel 6200 3350 3    50   Input ~ 0
+Text HLabel 4950 3300 2    50   Input ~ 0
 SDA
-Text HLabel 6300 3350 3    50   Input ~ 0
+Text HLabel 4950 3400 2    50   Input ~ 0
 SCL
-Text HLabel 5600 3350 3    50   Input ~ 0
+Text HLabel 4450 3600 0    50   Input ~ 0
 SD_SCK
-Text HLabel 5400 3350 3    50   Input ~ 0
+Text HLabel 4450 3400 0    50   Input ~ 0
 SD_DI
-Text HLabel 5500 3350 3    50   Input ~ 0
+Text HLabel 4450 3500 0    50   Input ~ 0
 SD_D0
-Text HLabel 5300 3350 3    50   Input ~ 0
+Text HLabel 4450 3300 0    50   Input ~ 0
 SD_SS
-Text HLabel 6100 3350 3    50   Input ~ 0
+Text HLabel 4950 3900 2    50   Input ~ 0
 TX
-Text HLabel 6000 3350 3    50   Input ~ 0
+Text HLabel 4950 3800 2    50   Input ~ 0
 Rx
-Text HLabel 7550 1350 0    50   Input ~ 0
+Text HLabel 7050 3600 2    50   Input ~ 0
 GND
-Text HLabel 8450 1350 2    50   Input ~ 0
+Text HLabel 7050 3400 2    50   Input ~ 0
 12V
 $Comp
-L power:GND #PWR049
+L power:GND #PWR051
 U 1 1 5FFF286B
-P 7700 1350
-F 0 "#PWR049" H 7700 1100 50  0001 C CNN
-F 1 "GND" H 7705 1177 50  0000 C CNN
-F 2 "" H 7700 1350 50  0001 C CNN
-F 3 "" H 7700 1350 50  0001 C CNN
-	1    7700 1350
+P 6950 3600
+F 0 "#PWR051" H 6950 3350 50  0001 C CNN
+F 1 "GND" H 6955 3427 50  0000 C CNN
+F 2 "" H 6950 3600 50  0001 C CNN
+F 3 "" H 6950 3600 50  0001 C CNN
+	1    6950 3600
+	1    0    0    -1
+$EndComp
+$Comp
+L power:+12V #PWR053
+U 1 1 5FFF3450
+P 6950 3400
+F 0 "#PWR053" H 6950 3250 50  0001 C CNN
+F 1 "+12V" H 6965 3573 50  0000 C CNN
+F 2 "" H 6950 3400 50  0001 C CNN
+F 3 "" H 6950 3400 50  0001 C CNN
+	1    6950 3400
 	1    0    0    -1
 $EndComp
 Wire Wire Line
-	7700 1350 7550 1350
+	6950 3400 7050 3400
 $Comp
-L power:+12V #PWR051
-U 1 1 5FFF3450
-P 8350 1350
-F 0 "#PWR051" H 8350 1200 50  0001 C CNN
-F 1 "+12V" H 8365 1523 50  0000 C CNN
-F 2 "" H 8350 1350 50  0001 C CNN
-F 3 "" H 8350 1350 50  0001 C CNN
-	1    8350 1350
+L power:GND #PWR048
+U 1 1 5FFF3FA3
+P 5400 3500
+F 0 "#PWR048" H 5400 3250 50  0001 C CNN
+F 1 "GND" H 5405 3327 50  0000 C CNN
+F 2 "" H 5400 3500 50  0001 C CNN
+F 3 "" H 5400 3500 50  0001 C CNN
+	1    5400 3500
 	-1   0    0    1
 $EndComp
-Wire Wire Line
-	8350 1350 8450 1350
 $Comp
-L power:GND #PWR046
-U 1 1 5FFF3FA3
-P 5700 3350
-F 0 "#PWR046" H 5700 3100 50  0001 C CNN
-F 1 "GND" H 5705 3177 50  0000 C CNN
-F 2 "" H 5700 3350 50  0001 C CNN
-F 3 "" H 5700 3350 50  0001 C CNN
-	1    5700 3350
+L power:+12V #PWR052
+U 1 1 5FFF43D1
+P 3850 3700
+F 0 "#PWR052" H 3850 3550 50  0001 C CNN
+F 1 "+12V" H 3865 3873 50  0000 C CNN
+F 2 "" H 3850 3700 50  0001 C CNN
+F 3 "" H 3850 3700 50  0001 C CNN
+	1    3850 3700
+	1    0    0    -1
+$EndComp
+Text HLabel 4450 3800 0    50   Input ~ 0
+SENSOR_VN
+Text HLabel 4450 3900 0    50   Input ~ 0
+SENSOR_VP
+$Comp
+L power:+3.3V #PWR049
+U 1 1 5FD44140
+P 5250 3700
+F 0 "#PWR049" H 5250 3550 50  0001 C CNN
+F 1 "+3.3V" H 5400 3750 50  0000 C CNN
+F 2 "" H 5250 3700 50  0001 C CNN
+F 3 "" H 5250 3700 50  0001 C CNN
+	1    5250 3700
 	1    0    0    -1
 $EndComp
 $Comp
-L power:+12V #PWR050
-U 1 1 5FFF43D1
-P 7700 3250
-F 0 "#PWR050" H 7700 3100 50  0001 C CNN
-F 1 "+12V" H 7715 3423 50  0000 C CNN
-F 2 "" H 7700 3250 50  0001 C CNN
-F 3 "" H 7700 3250 50  0001 C CNN
-	1    7700 3250
+L power:+5V #PWR050
+U 1 1 5FD44777
+P 4450 4000
+F 0 "#PWR050" H 4450 3850 50  0001 C CNN
+F 1 "+5V" H 4465 4173 50  0000 C CNN
+F 2 "" H 4450 4000 50  0001 C CNN
+F 3 "" H 4450 4000 50  0001 C CNN
+	1    4450 4000
+	0    -1   -1   0
+$EndComp
+$Comp
+L power:+3.3V #PWR055
+U 1 1 5FD45FA7
+P 6950 3100
+F 0 "#PWR055" H 6950 2950 50  0001 C CNN
+F 1 "+3.3V" H 6965 3273 50  0000 C CNN
+F 2 "" H 6950 3100 50  0001 C CNN
+F 3 "" H 6950 3100 50  0001 C CNN
+	1    6950 3100
 	1    0    0    -1
 $EndComp
 $Comp
-L Connector:Conn_01x16_Male J3
-U 1 1 5FD40501
-P 6100 3150
-F 0 "J3" V 5935 3078 50  0000 C CNN
-F 1 "Conn_01x16_Male" V 6026 3078 50  0000 C CNN
-F 2 "Connector_PinHeader_2.54mm:PinHeader_1x16_P2.54mm_Vertical_SMD_Pin1Left" H 6100 3150 50  0001 C CNN
-F 3 "~" H 6100 3150 50  0001 C CNN
-	1    6100 3150
-	0    1    1    0
+L power:+5V #PWR054
+U 1 1 5FD45FAD
+P 6950 2800
+F 0 "#PWR054" H 6950 2650 50  0001 C CNN
+F 1 "+5V" H 6965 2973 50  0000 C CNN
+F 2 "" H 6950 2800 50  0001 C CNN
+F 3 "" H 6950 2800 50  0001 C CNN
+	1    6950 2800
+	1    0    0    -1
 $EndComp
-Text HLabel 6400 3350 3    50   Input ~ 0
-SENSOR_VN
-Text HLabel 6500 3350 3    50   Input ~ 0
-SENSOR_VP
+Text HLabel 7050 2800 2    50   Input ~ 0
+5V
+Text HLabel 7050 3100 2    50   Input ~ 0
+3V3
 $Comp
-L power:+3.3V #PWR047
-U 1 1 5FD44140
-P 5800 3350
-F 0 "#PWR047" H 5800 3200 50  0001 C CNN
-F 1 "+3.3V" H 5815 3523 50  0000 C CNN
-F 2 "" H 5800 3350 50  0001 C CNN
-F 3 "" H 5800 3350 50  0001 C CNN
-	1    5800 3350
-	-1   0    0    1
-$EndComp
-$Comp
-L power:+5V #PWR048
-U 1 1 5FD44777
-P 6600 3350
-F 0 "#PWR048" H 6600 3200 50  0001 C CNN
-F 1 "+5V" H 6615 3523 50  0000 C CNN
-F 2 "" H 6600 3350 50  0001 C CNN
-F 3 "" H 6600 3350 50  0001 C CNN
-	1    6600 3350
-	-1   0    0    1
+L Connector_Generic:Conn_02x08_Odd_Even J3
+U 1 1 6007D5A3
+P 4650 3600
+F 0 "J3" H 4700 4117 50  0000 C CNN
+F 1 "Conn_02x08_Odd_Even" H 4700 4026 50  0000 C CNN
+F 2 "EZ-PY32:HTSS-108-01-YY-DV" H 4650 3600 50  0001 C CNN
+F 3 "~" H 4650 3600 50  0001 C CNN
+	1    4650 3600
+	1    0    0    -1
 $EndComp
 Wire Wire Line
-	6800 3350 7700 3350
+	4950 3700 5250 3700
 Wire Wire Line
-	7700 3350 7700 3250
-$Comp
-L power:+3.3V #PWR053
-U 1 1 5FD45FA7
-P 8550 1900
-F 0 "#PWR053" H 8550 1750 50  0001 C CNN
-F 1 "+3.3V" H 8565 2073 50  0000 C CNN
-F 2 "" H 8550 1900 50  0001 C CNN
-F 3 "" H 8550 1900 50  0001 C CNN
-	1    8550 1900
-	1    0    0    -1
-$EndComp
-$Comp
-L power:+5V #PWR052
-U 1 1 5FD45FAD
-P 8350 1900
-F 0 "#PWR052" H 8350 1750 50  0001 C CNN
-F 1 "+5V" H 8365 2073 50  0000 C CNN
-F 2 "" H 8350 1900 50  0001 C CNN
-F 3 "" H 8350 1900 50  0001 C CNN
-	1    8350 1900
-	1    0    0    -1
-$EndComp
-Text HLabel 8350 1900 0    50   Input ~ 0
-5V
-Text HLabel 8550 1900 2    50   Input ~ 0
-3V3
-NoConn ~ 5900 3350
-NoConn ~ 6700 3350
+	4450 3700 3850 3700
+Wire Wire Line
+	4950 3500 5400 3500
+NoConn ~ 4950 3600
+NoConn ~ 4950 4000
+Wire Wire Line
+	7050 2800 6950 2800
+Wire Wire Line
+	7050 3100 6950 3100
+Wire Wire Line
+	6950 3600 7050 3600
 $EndSCHEMATC
