File: Display.sch (KiCad schematic (older format))
At the start: 1 part, among them U2 3.5\"TFT_LCD_Shield

Commit message: Datenblätter hinzufügen und anschlüsse beschriften
Parts:
- added U?: PCF8574A, symbol Interface_Expansion:PCF8574A
- added U?: PCF8584, symbol Interface_Expansion:PCF8584
Changed lines of the file:
@@
 $Descr A4 11693 8268
 encoding utf-8
-Sheet 2 5
+Sheet 2 6
 Title ""
 Date ""
@@
 Wire Wire Line
 	4700 4150 4700 4350
+$Comp
+L Interface_Expansion:PCF8574A U?
+U 1 1 5FC808AE
+P 2500 3150
+F 0 "U?" H 2500 4031 50  0000 C CNN
+F 1 "PCF8574A" H 2500 3940 50  0000 C CNN
+F 2 "" H 2500 3150 50  0001 C CNN
+F 3 "http://www.nxp.com/documents/data_sheet/PCF8574_PCF8574A.pdf" H 2500 3150 50  0001 C CNN
+	1    2500 3150
+	1    0    0    -1
+$EndComp
+$Comp
+L Interface_Expansion:PCF8584 U?
+U 1 1 5FC821CA
+P 2550 5300
+F 0 "U?" H 2550 6481 50  0000 C CNN
+F 1 "PCF8584" H 2550 6390 50  0000 C CNN
+F 2 "" H 2550 5300 50  0001 C CNN
+F 3 "http://www.nxp.com/documents/data_sheet/PCF8584.pdf" H 2550 5300 50  0001 C CNN
+	1    2550 5300
+	-1   0    0    -1
+$EndComp
 $EndSCHEMATC

Commit message: i did everithing
Parts:
- removed U?: PCF8574A, symbol Interface_Expansion:PCF8574A
- removed U?: PCF8584, symbol Interface_Expansion:PCF8584
- renumbered U2 to U4
Connections:
- net 3V3 renamed +3V3
- net 5V renamed +5V
Changed lines of the file:
@@
 $Descr A4 11693 8268
 encoding utf-8
-Sheet 2 6
+Sheet 5 6
 Title ""
 Date ""
@@
 Text HLabel 5550 3800 2    50   Input ~ 0
 SC_SCK
-$Comp
-L ENCODER-RGB-SWITCH:3.5"TFT_LCD_Shield U2
-U 1 1 5FB3F30C
-P 4700 3150
-F 0 "U2" H 4100 4150 50  0000 C CNN
-F 1 "3.5\"TFT_LCD_Shield" H 5350 4150 50  0000 C CNN
-F 2 "EZ-PY32:kuman_display_3.5zoll" H 4300 3950 50  0001 C CNN
-F 3 "" H 4300 3950 50  0001 C CNN
-	1    4700 3150
-	1    0    0    -1
-$EndComp
 Wire Wire Line
 	3900 2750 4100 2750
@@
 	3900 3450 4100 3450
 Wire Wire Line
-	4600 2200 4600 2350
+	4600 2200 4600 2250
 Wire Wire Line
-	4800 2200 4800 2350
+	4800 2200 4800 2250
 Wire Wire Line
 	5350 2750 5500 2750
@@
 	4700 4150 4700 4350
 $Comp
-L Interface_Expansion:PCF8574A U?
-U 1 1 5FC808AE
-P 2500 3150
-F 0 "U?" H 2500 4031 50  0000 C CNN
-F 1 "PCF8574A" H 2500 3940 50  0000 C CNN
-F 2 "" H 2500 3150 50  0001 C CNN
-F 3 "http://www.nxp.com/documents/data_sheet/PCF8574_PCF8574A.pdf" H 2500 3150 50  0001 C CNN
-	1    2500 3150
+L ENCODER-RGB-SWITCH:3.5"TFT_LCD_Shield U4
+U 1 1 5FB3F30C
+P 4700 3150
+F 0 "U4" H 4100 4150 50  0000 C CNN
+F 1 "3.5\"TFT_LCD_Shield" H 5350 4150 50  0000 C CNN
+F 2 "EZ-PY32:kuman_display_3.5zoll" H 4300 3950 50  0001 C CNN
+F 3 "" H 4300 3950 50  0001 C CNN
+	1    4700 3150
 	1    0    0    -1
 $EndComp
 $Comp
-L Interface_Expansion:PCF8584 U?
-U 1 1 5FC821CA
-P 2550 5300
-F 0 "U?" H 2550 6481 50  0000 C CNN
-F 1 "PCF8584" H 2550 6390 50  0000 C CNN
-F 2 "" H 2550 5300 50  0001 C CNN
-F 3 "http://www.nxp.com/documents/data_sheet/PCF8584.pdf" H 2550 5300 50  0001 C CNN
-	1    2550 5300
-	-1   0    0    -1
+L power:+3.3V #PWR045
+U 1 1 5FFBB000
+P 5900 2100
+F 0 "#PWR045" H 5900 1950 50  0001 C CNN
+F 1 "+3.3V" H 5915 2273 50  0000 C CNN
+F 2 "" H 5900 2100 50  0001 C CNN
+F 3 "" H 5900 2100 50  0001 C CNN
+	1    5900 2100
+	1    0    0    -1
 $EndComp
+Wire Wire Line
+	5900 2100 5900 2250
+Wire Wire Line
+	5900 2250 4800 2250
+Connection ~ 4800 2250
+Wire Wire Line
+	4800 2250 4800 2350
+$Comp
+L power:+5V #PWR044
+U 1 1 5FFBBB03
+P 4050 1850
+F 0 "#PWR044" H 4050 1700 50  0001 C CNN
+F 1 "+5V" H 4065 2023 50  0000 C CNN
+F 2 "" H 4050 1850 50  0001 C CNN
+F 3 "" H 4050 1850 50  0001 C CNN
+	1    4050 1850
+	1    0    0    -1
+$EndComp
+Wire Wire Line
+	4050 2250 4050 1850
+Wire Wire Line
+	4050 2250 4600 2250
+Connection ~ 4600 2250
+Wire Wire Line
+	4600 2250 4600 2350
 $EndSCHEMATC

Commit message: Add CAD
Parts:
- renumbered U4 to U6
Changed lines of the file:
@@
 	4700 4150 4700 4350
 $Comp
-L ENCODER-RGB-SWITCH:3.5"TFT_LCD_Shield U4
+L ENCODER-RGB-SWITCH:3.5"TFT_LCD_Shield U6
 U 1 1 5FB3F30C
 P 4700 3150
-F 0 "U4" H 4100 4150 50  0000 C CNN
+F 0 "U6" H 4100 4150 50  0000 C CNN
 F 1 "3.5\"TFT_LCD_Shield" H 5350 4150 50  0000 C CNN
 F 2 "EZ-PY32:kuman_display_3.5zoll" H 4300 3950 50  0001 C CNN
@@
 $EndComp
 $Comp
-L power:+3.3V #PWR045
+L power:+3.3V #PWR047
 U 1 1 5FFBB000
 P 5900 2100
-F 0 "#PWR045" H 5900 1950 50  0001 C CNN
+F 0 "#PWR047" H 5900 1950 50  0001 C CNN
 F 1 "+3.3V" H 5915 2273 50  0000 C CNN
 F 2 "" H 5900 2100 50  0001 C CNN
@@
 	4800 2250 4800 2350
 $Comp
-L power:+5V #PWR044
+L power:+5V #PWR046
 U 1 1 5FFBBB03
 P 4050 1850
-F 0 "#PWR044" H 4050 1700 50  0001 C CNN
+F 0 "#PWR046" H 4050 1700 50  0001 C CNN
 F 1 "+5V" H 4065 2023 50  0000 C CNN
 F 2 "" H 4050 1850 50  0001 C CNN
