File: Drehencoder.sch (KiCad schematic (older format))
At the start: 1 part

Commit message: Datenblätter hinzufügen und anschlüsse beschriften
Parts:
- added C?: 0.01uF, symbol Device:C
- added C? (x2): C, symbol Device:C
- added R? (x4): 10k, symbol Device:R
- added R? (x2): R, symbol Device:R
- added SW?: SW_Push, symbol Switch:SW_Push
Connections:
- net Potti_A: now also C?.2, R?.1; no longer S1.A
- net Potti_B: now also C?.2, R?.2; no longer S1.B
- net Potti_C renamed GND
- net GND: now also C?.1, C?.1, C?.2, SW?.2
- net vcc? renamed +5V
- net +5V: now also R?.1, R?.2, R?.2
- new net: R?.1, R?.2, S1.A
- new net: R?.1, R?.1, S1.B
- new net: C?.1, R?.1, R?.2
- new net: R?.2, SW?.1

Commit message: i did everithing
Parts:
- removed R?: R, symbol Device:R
- removed SW?: SW_Push, symbol Switch:SW_Push
- added Q1, Q2, Q3: DTC144E, Package_TO_SOT_SMD:SOT-23, symbol Transistor_BJT:DTC144E
- added R5: 120R, Resistor_SMD:R_0603_1608Metric_Pad0.98x0.95mm_HandSolder, symbol Device:R
- added R6, R7: 68R, Resistor_SMD:R_0603_1608Metric_Pad0.98x0.95mm_HandSolder, symbol Device:R
- added R9: 94k, Resistor_SMD:R_0603_1608Metric_Pad0.98x0.95mm_HandSolder, symbol Device:R
- C1: renamed from C?; value 0.01uF -> 10nF; footprint (none) -> Capacitor_SMD:C_0603_1608Metric_Pad1.08x0.95mm_HandSolder
- C2, C3: renamed from C?; value C -> 10nF; footprint (none) -> Capacitor_SMD:C_0603_1608Metric_Pad1.08x0.95mm_HandSolder
- R1, R2, R3, R4: renamed from R?; footprint (none) -> Resistor_SMD:R_0603_1608Metric_Pad0.98x0.95mm_HandSolder
- R8: renamed from R?; value R -> 47k; footprint (none) -> Resistor_SMD:R_0603_1608Metric_Pad0.98x0.95mm_HandSolder
Connections:
- net GND: now also Q1.2 (E), Q2.2 (E), Q3.2 (E), R9.2
- net schalter_masse: now also C3.1, R8.1, R9.1; no longer S1.3
- net at R8.2: now also S1.3
- net Rot_masse: no longer names the net of S1.1
- net Rot_masse: now also R5.2
- net blau_masse: no longer names the net of S1.4
- net blau_masse: now also R7.2
- net gruen_masse: no longer names the net of S1.2
- net gruen_masse: now also R6.2
- new net: Q3.3 (C), R5.1
- new net: Q2.3 (C), R6.1
- new net: Q1.3 (C), R7.1
- new net blau: Q1.1 (B)
- new net gruen: Q2.1 (B)
- new net rot: Q3.1 (B)
Other:
- moved on the sheet: C3, R8

Commit message: Add CAD
Parts:
- R9: value 94k -> 100k
Connections:
- net Potti_A renamed Encoder_A
- net Potti_B renamed Encoder_B
Changed lines of the file:
@@
 	1    0    0    -1
 $EndComp
-Text HLabel 4200 2700 0    50   Input ~ 0
-Potti_A
 Text HLabel 4200 4550 0    50   Input ~ 0
-Potti_B
+Encoder_B
 Text HLabel 6400 4400 0    50   Input ~ 0
 rot
@@
 P 8350 4450
 F 0 "R9" H 8420 4496 50  0000 L CNN
-F 1 "94k" H 8420 4405 50  0000 L CNN
+F 1 "100k" H 8420 4405 50  0000 L CNN
 F 2 "Resistor_SMD:R_0603_1608Metric_Pad0.98x0.95mm_HandSolder" V 8280 4450 50  0001 C CNN
 F 3 "~" H 8350 4450 50  0001 C CNN
@@
 Wire Wire Line
 	8350 4600 8350 4850
+Text HLabel 4200 2700 0    50   Input ~ 0
+Encoder_A
 $EndSCHEMATC
