File: ESP32.sch (KiCad schematic (older format))
At the start: 12 parts

Commit message: i did everithing
Parts:
- removed C?: 100nF, symbol Device:C
- removed U?: ESP32-WROOM-32U, RF_Module:ESP32-WROOM-32U, symbol RF_Module:ESP32-WROOM-32U
- added C9: 1u, Capacitor_SMD:C_0603_1608Metric_Pad1.08x0.95mm_HandSolder, symbol Device:C
- added J2: Conn_01x06_Male, Connector_PinHeader_2.54mm:PinHeader_1x06_P2.54mm_Horizontal, symbol Connector:Conn_01x06_Male
- added Q4: Q_PNP_BCE, Package_TO_SOT_SMD:SOT-23, symbol Device:Q_PNP_BCE
- added Q5: BC847BW_135, Package_TO_SOT_SMD:SOT-323_SC-70, symbol Device:Q_NPN_BEC
- added R12, R13, R16, R17: 10k, Resistor_SMD:R_0603_1608Metric_Pad0.98x0.95mm_HandSolder, symbol Device:R
- added U3: ESP32-WROOM-32, RF_Module:ESP32-WROOM-32, symbol RF_Module:ESP32-WROOM-32
- C10: renamed from C?; value 10uF -> 22uF; footprint (none) -> Capacitor_SMD:C_0603_1608Metric_Pad1.08x0.95mm_HandSolder
- C11: renamed from C?; footprint (none) -> Capacitor_SMD:C_0603_1608Metric_Pad1.08x0.95mm_HandSolder
- C7, C8: renamed from C?; value C -> 1uF; footprint (none) -> Capacitor_SMD:C_0603_1608Metric_Pad1.08x0.95mm_HandSolder
- R10, R14: renamed from R?; value R -> 100k; footprint (none) -> Resistor_SMD:R_0603_1608Metric_Pad0.98x0.95mm_HandSolder
- R11, R15: renamed from R?; value R -> 470k; footprint (none) -> Resistor_SMD:R_0603_1608Metric_Pad0.98x0.95mm_HandSolder
- SW1, SW2: renamed from SW?; footprint (none) -> Button_Switch_SMD:SW_SPST_B3U-1000P
Connections:
- net labels added: DTR, Potti_A, Potti_B, Potti_schalter, RTS, Rx, Rx_stecker, SCL, SDA, SENSOR_VN, SENSOR_VP, Tx, blau, gruen, rot
- net labels removed: SC_SCK, SD_D0, SD_DI, SD_SS
- wire segments 54 -> 90
- no-connect marks 0 -> 7
Other:
- note added: "Auto Programm Circuit\n-----------------\nDTR RTS RST GPIO0\n1 | 1 | 1 | 1\n0 | 0 | 1 | 1\n1 | 0 | 0 | 1\n0 | 1 | 1 | 0"
- note added: "ESP32-WROOM-32U Modul\n\n"
- note added: "Logikschaltung für \nautomatischen Bootvorgang"
- note added: "R & C Werte\nnoch ermitteln"
- note added: "RC Glied ensure power supply during power-up"
- note added: "UART Programmierbar"
- note added: "laut datenblatt NC"
- note added: "mit externem Antennenanschluß"
- moved on the sheet: C11

Commit message: smal fixes
Connections:
- net LCD_RS: now also U3.37 (IO23); no longer U3.6 (IO34)
- net LCD_WR: now also U3.36 (IO22); no longer U3.7 (IO35)
- net Potti_A: now also U3.7 (IO35); no longer U3.37 (IO23)
- net Potti_B: now also U3.6 (IO34); no longer U3.36 (IO22)
Changed lines of the file:
@@
 Wire Wire Line
 	6900 4850 6700 4850
-Text HLabel 6900 5050 2    50   Input ~ 0
+Text HLabel 6900 4250 2    50   Input ~ 0
 LCD_WR
 Text HLabel 6900 4750 2    50   Input ~ 0
@@
 Text HLabel 6900 4050 2    50   Input ~ 0
 LCD_CS
-Text HLabel 6900 4950 2    50   Input ~ 0
+Text HLabel 6900 4350 2    50   Input ~ 0
 LCD_RS
 Text HLabel 6900 4150 2    50   Input ~ 0
@@
 Wire Wire Line
 	6700 3850 6900 3850
-Text HLabel 6900 4250 2    50   Input ~ 0
+Text HLabel 6900 4950 2    50   Input ~ 0
 Potti_B
-Text HLabel 6900 4350 2    50   Input ~ 0
+Text HLabel 6900 5050 2    50   Input ~ 0
 Potti_A
 NoConn ~ 5500 3950

Commit message: Add CAD
Parts:
- added R17, R19: 4k7, Resistor_SMD:R_0603_1608Metric_Pad0.98x0.95mm_HandSolder, symbol Device:R
- renumbered R17 to R18, U3 to U5
Connections:
- net +3V3: now also R17.1, R19.1
- net SCL: now also R17.2
- net SDA: now also R19.2
- net Potti_A renamed Encoder_A
- net Potti_B renamed Encoder_B
- net Potti_schalter renamed Encoder_schalter
Other:
- note added: "I^2C"
Changed lines of the file:
@@
 LCD_RST
-Wire Wire Line
-	6700 3250 6900 3250
 Wire Wire Line
 	6700 4050 6900 4050
@@
 	4400 1700 4150 1700
 Connection ~ 4400 1700
-Text HLabel 9000 3800 0    50   Input ~ 0
+Text HLabel 7100 5500 0    50   Input ~ 0
 GND
 Text GLabel 7550 2850 2    50   Input ~ 0
@@
 	7550 3050 7450 3050
 Wire Wire Line
-	6900 3350 6700 3350
-Wire Wire Line
 	6900 3450 6700 3450
 Text HLabel 7800 2700 2    50   Input ~ 0
@@
 blau
 Text HLabel 6900 4450 2    50   Input ~ 0
-Potti_schalter
-Wire Wire Line
-	6900 3950 6700 3950
+Encoder_schalter
 Wire Wire Line
 	6900 3150 6700 3150
@@
 	6700 3850 6900 3850
 Text HLabel 6900 4950 2    50   Input ~ 0
-Potti_B
+Encoder_B
 Text HLabel 6900 5050 2    50   Input ~ 0
-Potti_A
+Encoder_A
 NoConn ~ 5500 3950
 NoConn ~ 5500 4050
@@
 Text Notes 5400 4550 1    50   ~ 0
 laut datenblatt NC
-Wire Wire Line
-	6700 4550 6900 4550
 Text Notes 4900 3450 0    50   ~ 0
 R & C Werte\nnoch ermitteln
@@
 Wire Wire Line
 	6700 2750 6950 2750
-Text HLabel 6900 3250 2    50   Input ~ 0
+Text HLabel 7900 3450 2    50   Input ~ 0
 SDA
-Text HLabel 6900 3950 2    50   Input ~ 0
+Text HLabel 7950 3750 2    50   Input ~ 0
 SCL
 NoConn ~ 3700 400
@@
 	6100 5350 6100 5500
 $Comp
-L power:GND #PWR043
+L power:GND #PWR045
 U 1 1 5FFCB3AE
-P 9100 3950
-F 0 "#PWR043" H 9100 3700 50  0001 C CNN
-F 1 "GND" H 9105 3777 50  0000 C CNN
-F 2 "" H 9100 3950 50  0001 C CNN
-F 3 "" H 9100 3950 50  0001 C CNN
-	1    9100 3950
-	1    0    0    -1
-$EndComp
-Wire Wire Line
-	9000 3800 9100 3800
-Wire Wire Line
-	9100 3800 9100 3950
+P 7200 5650
+F 0 "#PWR045" H 7200 5400 50  0001 C CNN
+F 1 "GND" H 7205 5477 50  0000 C CNN
+F 2 "" H 7200 5650 50  0001 C CNN
+F 3 "" H 7200 5650 50  0001 C CNN
+	1    7200 5650
+	1    0    0    -1
+$EndComp
+Wire Wire Line
+	7100 5500 7200 5500
+Wire Wire Line
+	7200 5500 7200 5650
 Text HLabel 5500 3050 0    50   Input ~ 0
 SENSOR_VN
@@
 	2200 4050 2200 4300
 $Comp
-L Device:R R17
+L Device:R R18
 U 1 1 5FD60A3E
 P 8150 2950
-F 0 "R17" V 7943 2950 50  0000 C CNN
+F 0 "R18" V 7943 2950 50  0000 C CNN
 F 1 "10k" V 8034 2950 50  0000 C CNN
 F 2 "Resistor_SMD:R_0603_1608Metric_Pad0.98x0.95mm_HandSolder" V 8080 2950 50  0001 C CNN
@@
 	7450 2950 8000 2950
 $Comp
-L RF_Module:ESP32-WROOM-32 U3
+L RF_Module:ESP32-WROOM-32 U5
 U 1 1 5FD79442
 P 6100 3950
-F 0 "U3" H 6100 5531 50  0000 C CNN
+F 0 "U5" H 6100 5531 50  0000 C CNN
 F 1 "ESP32-WROOM-32" H 6100 5440 50  0000 C CNN
 F 2 "RF_Module:ESP32-WROOM-32" H 6100 2450 50  0001 C CNN
@@
 Text Notes 3900 2400 0    50   ~ 0
 RC Glied ensure power supply during power-up
+Wire Wire Line
+	6700 3250 7850 3250
+Wire Wire Line
+	7850 3250 7850 3450
+Wire Wire Line
+	7850 3450 7900 3450
+Wire Wire Line
+	7850 3250 8200 3250
+Connection ~ 7850 3250
+$Comp
+L Device:R R19
+U 1 1 5FF83538
+P 8350 3250
+F 0 "R19" V 8143 3250 50  0000 C CNN
+F 1 "4k7" V 8234 3250 50  0000 C CNN
+F 2 "Resistor_SMD:R_0603_1608Metric_Pad0.98x0.95mm_HandSolder" V 8280 3250 50  0001 C CNN
+F 3 "~" H 8350 3250 50  0001 C CNN
+	1    8350 3250
+	0    1    1    0
+$EndComp
+$Comp
+L Device:R R17
+U 1 1 5FF83E9C
+P 8350 3950
+F 0 "R17" H 8420 3996 50  0000 L CNN
+F 1 "4k7" H 8420 3905 50  0000 L CNN
+F 2 "Resistor_SMD:R_0603_1608Metric_Pad0.98x0.95mm_HandSolder" V 8280 3950 50  0001 C CNN
+F 3 "~" H 8350 3950 50  0001 C CNN
+	1    8350 3950
+	0    1    1    0
+$EndComp
+$Comp
+L power:+3.3V #PWR044
+U 1 1 5FF8446D
+P 8650 3250
+F 0 "#PWR044" H 8650 3100 50  0001 C CNN
+F 1 "+3.3V" H 8665 3423 50  0000 C CNN
+F 2 "" H 8650 3250 50  0001 C CNN
+F 3 "" H 8650 3250 50  0001 C CNN
+	1    8650 3250
+	1    0    0    -1
+$EndComp
+$Comp
+L power:+3.3V #PWR043
+U 1 1 5FF84C5E
+P 8650 3750
+F 0 "#PWR043" H 8650 3600 50  0001 C CNN
+F 1 "+3.3V" H 8665 3923 50  0000 C CNN
+F 2 "" H 8650 3750 50  0001 C CNN
+F 3 "" H 8650 3750 50  0001 C CNN
+	1    8650 3750
+	1    0    0    -1
+$EndComp
+Wire Wire Line
+	8500 3250 8650 3250
+Wire Wire Line
+	6700 3350 6900 3350
+Wire Wire Line
+	6700 4550 6900 4550
+Wire Wire Line
+	8650 3950 8500 3950
+Wire Wire Line
+	8650 3750 8650 3950
+Wire Wire Line
+	6700 3950 7850 3950
+Wire Wire Line
+	7950 3750 7850 3750
+Wire Wire Line
+	7850 3750 7850 3950
+Connection ~ 7850 3950
+Wire Wire Line
+	7850 3950 8200 3950
+Text Notes 7950 3650 0    50   ~ 0
+I^2C
 $EndSCHEMATC
