File: EZ-PY32.sch (KiCad schematic (older format))
At the start: 1 part, among them U1 ESP32-WROOM-32U

Commit message: Datenblätter hinzufügen und anschlüsse beschriften
Parts:
- removed U1: ESP32-WROOM-32U, RF_Module:ESP32-WROOM-32U, symbol RF_Module:ESP32-WROOM-32U
Connections:
- net labels added: +12V, +3.3V, +5V, GND
- wire segments 0 -> 20

Commit message: i did everithing
Parts:
- added H1, H2, H3, H4: MountingHole, MountingHole:MountingHole_3.5mm, symbol Mechanical:MountingHole
Connections:
- net labels added: LCD_CS, LCD_RD, LCD_RS, LCD_RST, LCD_WR, Rx_extern, SD_D0, SD_DI, SD_SCK, SD_SS, SENSOR_VN, SENSOR_VP, Tx_extern
- wire segments 20 -> 90

Commit message: smal fixes
Parts:
- added U5: OTH_LOGO, EZ-PY32:OTH_3000x3000dpi, symbol ENCODER-RGB-SWITCH:OTH_LOGO
- added U6: EZ-PY32LOGO, EZ-PY32:EZ, symbol ENCODER-RGB-SWITCH:EZ-PY32LOGO
Changed lines of the file:
@@
+	1    0    0    -1
+$EndComp
+$Comp
+L ENCODER-RGB-SWITCH:EZ-PY32LOGO U6
+U 1 1 5FF77B7E
+P 4650 1000
+F 0 "U6" H 4650 1215 50  0000 C CNN
+F 1 "EZ-PY32LOGO" H 4650 1124 50  0000 C CNN
+F 2 "EZ-PY32:EZ" H 4650 1000 50  0001 C CNN
+F 3 "" H 4650 1000 50  0001 C CNN
+	1    4650 1000
+	1    0    0    -1
+$EndComp
+$Comp
+L ENCODER-RGB-SWITCH:OTH_LOGO U5
+U 1 1 5FF77F48
+P 4550 1350
+F 0 "U5" H 4550 1565 50  0000 C CNN
+F 1 "OTH_LOGO" H 4550 1474 50  0000 C CNN
+F 2 "EZ-PY32:OTH_3000x3000dpi" H 4550 1350 50  0001 C CNN
+F 3 "" H 4550 1350 50  0001 C CNN
+	1    4550 1350
 	1    0    0    -1
 $EndComp

Commit message: Add CAD
Parts:
- renumbered U5 to U1, U6 to U2
Changed lines of the file:
@@
 F0 "Drehencoder" 50
 F1 "Drehencoder.sch" 50
-F2 "Potti_A" I L 8100 3700 50
-F3 "Potti_B" I L 8100 3850 50
+F2 "Encoder_A" I L 8100 3700 50
+F3 "Encoder_B" I L 8100 3850 50
 F4 "schalter_masse" I L 8100 4000 50
 F5 "5V" I R 9300 3350 50
@@
 F16 "GND" I L 5350 6400 50
 F17 "Tx" I R 6550 3150 50
-F18 "Potti_A" I R 6550 4050 50
-F19 "Potti_B" I R 6550 4200 50
+F18 "Encoder_A" I R 6550 4050 50
+F19 "Encoder_B" I R 6550 4200 50
 F20 "rot" I R 6550 4650 50
 F21 "gruen" I R 6550 4950 50
 F22 "blau" I R 6550 4800 50
-F23 "Potti_schalter" I R 6550 4350 50
+F23 "Encoder_schalter" I R 6550 4350 50
 F24 "SDA" I L 5350 3250 50
 F25 "SCL" I L 5350 3400 50
@@
 $EndComp
 $Comp
-L ENCODER-RGB-SWITCH:EZ-PY32LOGO U6
+L ENCODER-RGB-SWITCH:EZ-PY32LOGO U2
 U 1 1 5FF77B7E
 P 4650 1000
-F 0 "U6" H 4650 1215 50  0000 C CNN
+F 0 "U2" H 4650 1215 50  0000 C CNN
 F 1 "EZ-PY32LOGO" H 4650 1124 50  0000 C CNN
 F 2 "EZ-PY32:EZ" H 4650 1000 50  0001 C CNN
@@
 $EndComp
 $Comp
-L ENCODER-RGB-SWITCH:OTH_LOGO U5
+L ENCODER-RGB-SWITCH:OTH_LOGO U1
 U 1 1 5FF77F48
 P 4550 1350
-F 0 "U5" H 4550 1565 50  0000 C CNN
+F 0 "U1" H 4550 1565 50  0000 C CNN
 F 1 "OTH_LOGO" H 4550 1474 50  0000 C CNN
 F 2 "EZ-PY32:OTH_3000x3000dpi" H 4550 1350 50  0001 C CNN
